File: PCB/deskrgbm.kicad_sch (KiCad schematic)
At the start: 130 parts, among them SW1 RotaryEncoder_Switch_MP, U1 XIAO-RP2040-DIP

Commit message: Journal + CAD
Parts:
- C1, C10, C11, C12, C13, C14, C15, C16, C17, C18, C19, C2, C20, C21, C22, C23, C24, C25, C26, C27, C28, C29, C3, C30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: footprint Capacitor_SMD:C_0402_1005Metric -> Capacitor_THT:C_Disc_D3.0mm_W1.6mm_P2.50mm
